Commit message: moved lidar

File: bamboomba_description/urdf/sensors.urdf.xacro (robot description, xacro)
@@ -6,5 +6,5 @@
     <inertial>
       <mass value="0.001"/>
-      <origin xyz="0 0 0" rpy="0 0 ${pi/2}"/>
+      <origin xyz="0 0 0" rpy="0 0 0"/>
       <inertia ixx="${dummy_inertia}" ixy="0.0" ixz="0.0" iyy="${dummy_inertia}" iyz="0.0" izz="${dummy_inertia}"/>
     </inertial>
@@ -25,5 +25,8 @@
     <parent link="base_link"/>
     <child link="base_scan" />
-    <origin xyz="-0.035 0.0 0.082" rpy="0 0 ${pi+pi/4}" />
+    <!-- Bottom platform -->
+    <!--<origin xyz="-0.035 0.0 0.082" rpy="0 0 0" />-->
+    <!-- Top platform -->
+    <origin xyz="0.0 0.0 0.254" rpy="0 0 ${pi}" />
   </joint>
   <!-- RGBD Camera -->
